File: pcb/jackalope_unibody.kicad_pcb (KiCad board)
At the start: 2 copper layers, 347.5 x 155.4 mm, 101 parts

Commit message: pcb getting prettier
Parts:
- added G***: LOGO, jackalope:bighornFP, F.Cu at (150.0, 19.2)
- added G***: LOGO, jackalope:bighornFP, F.Cu at (148.8, 12.2)
- added G***: LOGO, jackalope:bighornFP, F.Cu at (144.5, 7.75)
- added G***: LOGO, jackalope:bighornFP, F.Cu at (149.5, 10.2)
Other:
- board text added: "Jackalope unibody v1.0 by HBBisenieks"

Commit message: begin split work, spelling mistake fixed, gerbers
Parts:
- added RESET: SW_PUSH, Keebio-Parts:SW_Tactile_SPST_Angled_MJTP1117, F.Cu at (189.2, -41.5)
Routing:
- net RST: track 0.00 -> 42.6 mm
- net GND: track 18.8 -> 55.4 mm
Changed lines of the file:
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@@
     (thickness 1.6)
     (drawings 80)
-    (tracks 733)
+    (tracks 740)
     (zones 0)
-    (modules 105)
+    (modules 106)
     (nets 73)
   )
@@
     (add_net ring_top)
   )
+  (module Keebio-Parts:SW_Tactile_SPST_Angled_MJTP1117 (layer F.Cu)
+    (at 189.25 -41.5)
+    (descr "tactile switch SPST right angle, PTS645VL39-2 LFS")
+    (tags "tactile switch SPST angled PTS645VL39-2 LFS C&K Button")
+    (fp_text reference RESET (at 2.5 1.68) (layer F.SilkS)
+      (effects (font (size 1 1) (thickness 0.15)))
+    )
+    (fp_text value SW_PUSH (at 2.5 5.38988) (layer F.Fab)
+      (effects (font (size 1 1) (thickness 0.15)))
+    )
+    (fp_line (start 0.8 0.97) (end 4.2 0.97) (layer F.SilkS) (width 0.12))
+    (fp_line (start -0.84 0.97) (end -0.3 0.97) (layer F.SilkS) (width 0.12))
+    (fp_line (start 5.3 0.97) (end 5.84 0.97) (layer F.SilkS) (width 0.12))
+    (fp_line (start 5.84 0.97) (end 5.84 1.2) (layer F.SilkS) (width 0.12))
+    (fp_line (start -0.95 3.6) (end -0.95 0.86) (layer F.Fab) (width 0.1))
+    (fp_line (start 5.95 3.6) (end 6.25 3.6) (layer F.Fab) (width 0.1))
+    (fp_line (start -1.25 3.6) (end -1.25 -2.59) (layer F.Fab) (width 0.1))
+    (fp_line (start -1.25 -2.59) (end 6.25 -2.59) (layer F.Fab) (width 0.1))
+    (fp_line (start -1.36 -2.7) (end -1.36 1.2) (layer F.SilkS) (width 0.12))
+    (fp_line (start 6.36 -2.7) (end 6.36 1.2) (layer F.SilkS) (width 0.12))
+    (fp_line (start -1.36 -2.7) (end 6.36 -2.7) (layer F.SilkS) (width 0.12))
+    (fp_line (start -2.25 4.45) (end -2.25 -2.8) (layer F.CrtYd) (width 0.05))
+    (fp_line (start 7.3 4.45) (end -2.25 4.45) (layer F.CrtYd) (width 0.05))
+    (fp_line (start 7.3 -2.8) (end 7.3 4.45) (layer F.CrtYd) (width 0.05))
+    (fp_line (start -2.25 -2.8) (end 7.3 -2.8) (layer F.CrtYd) (width 0.05))
+    (fp_line (start 6.25 3.6) (end 6.25 -2.59) (layer F.Fab) (width 0.1))
+    (fp_line (start -0.95 0.86) (end 5.95 0.86) (layer F.Fab) (width 0.1))
+    (fp_line (start -1.25 3.6) (end -0.95 3.6) (layer F.Fab) (width 0.1))
+    (fp_line (start 5.95 3.6) (end 5.95 0.86) (layer F.Fab) (width 0.1))
+    (fp_line (start -0.84 0.97) (end -0.84 1.2) (layer F.SilkS) (width 0.12))
+    (fp_line (start 1.05 -3.85) (end 3.95 -3.85) (layer F.Fab) (width 0.1))
+    (fp_line (start 3.95 -3.85) (end 3.95 -2.59) (layer F.Fab) (width 0.1))
+    (fp_line (start 1.05 -3.85) (end 1.05 -2.59) (layer F.Fab) (width 0.1))
+    (pad "" np_thru_hole circle (at 2.5 -1.21) (size 1.2 1.2) (drill 1.2) (layers *.Cu *.Mask))
+    (pad "" thru_hole circle (at -1 2.49) (size 2.1 2.1) (drill 1.3) (layers *.Cu *.Mask))
+    (pad 1 thru_hole circle (at 0 0) (size 1.75 1.75) (drill 0.99) (layers *.Cu *.Mask)
+      (net 70 GND))
+    (pad 2 thru_hole circle (at 5 0) (size 1.75 1.75) (drill 0.99) (layers *.Cu *.Mask)
+      (net 71 RST))
+    (pad "" thru_hole circle (at 6.01 2.49) (size 2.1 2.1) (drill 1.3) (layers *.Cu *.Mask))
+    (model ${KISYS3DMOD}/Buttons_Switches_THT.3dshapes/SW_Tactile_SPST_Angled_PTS645Vx39-2LFS.wrl
+      (at (xyz 0 0 0))
+      (scale (xyz 1 1 1))
+      (rotate (xyz 0 0 0))
+    )
+  )
   (module jackalope:bighornFP (layer F.Cu)
     (at 150 19.25)
@@
   (segment (start 155.879315 -25.184852) (end 158.419315 -27.724852) (width 0.25) (layer B.Cu) (net 70))
   (segment (start 143.179315 -25.184852) (end 155.879315 -25.184852) (width 0.25) (layer B.Cu) (net 70))
+  (segment (start 189.25 -41.5) (end 187.5 -41.5) (width 0.25) (layer F.Cu) (net 70))
+  (segment (start 187.5 -41.5) (end 183.75 -37.75) (width 0.25) (layer F.Cu) (net 70))
+  (segment (start 168.444463 -37.75) (end 158.419315 -27.724852) (width 0.25) (layer F.Cu) (net 70))
+  (segment (start 183.75 -37.75) (end 168.444463 -37.75) (width 0.25) (layer F.Cu) (net 70))
+  (segment (start 168.634482 -35.400019) (end 158.419315 -25.184852) (width 0.25) (layer F.Cu) (net 71))
+  (segment (start 188.150019 -35.400019) (end 168.634482 -35.400019) (width 0.25) (layer F.Cu) (net 71))
+  (segment (start 194.25 -41.5) (end 188.150019 -35.400019) (width 0.25) (layer F.Cu) (net 71))
 )
