File: pcb/v2_0/monoblock/jackalope_unibody.kicad_pcb (KiCad board)
At the start: 2 copper layers, 329.5 x 134.9 mm, 153 parts

Commit message: update pcb file
Other:
- board text added: "Jackalope Keyboard v2.0 by @HBBisenieks"
- board text removed: "Jackalope Keyboard by @HBBisenieks"
Changed lines of the file:
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@@
       (outputformat 1)
       (mirror false)
-      (drillshape 1)
+      (drillshape 0)
       (scaleselection 1)
-      (outputdirectory ""))
+      (outputdirectory "jacalope_unibody_gerbers/"))
   )
   (net 0 "")
@@
       (net 3 P9))
   )
-  (gr_text "Jackalope Keyboard by @HBBisenieks" (at 49.5 19 -15) (layer B.Cu)
+  (gr_text "Jackalope Keyboard v2.0 by @HBBisenieks" (at 49.5 19 -15) (layer B.Cu)
     (effects (font (size 1.5 1.5) (thickness 0.3)))
   )
