File: pcb/v2_0/split/jackalope_split.kicad_pcb (KiCad board)
At the start: 2 copper layers, 171.9 x 116.3 mm, 81 parts

Commit message: split pcb routed, gerbers
Parts:
- moved G*** 2.02 mm to (67.2, -26.8)
- moved RESET 1.27 mm to (137.5, -13.5)
- moved G*** 1.12 mm to (63.8, -27.0)
Connections:
- MCU1 pad 15: Reset_GND -> GND
- MCU1 pad 16: Reset_GND -> GND
- MCU1 pad 2: Reset_GND -> GND
- MCU2 pad 15: Reset_GND -> GND
- MCU2 pad 16: Reset_GND -> GND
- MCU2 pad 2: Reset_GND -> GND
- REF** pad 3: Reset_GND -> GND
- RESET pad 2: Reset_GND -> (no net)
Routing:
- net GND: track 0.00 -> 109.5 mm, vias 0 -> 1
- net Reset_GND: track 71.3 -> 0.00 mm
- net P3: track 210.0 -> 278.6 mm, vias 3 -> 2
- net P5: track 176.6 -> 234.2 mm
- net P4: track 204.4 -> 240.3 mm
- net P0: track 206.4 -> 238.1 mm
- net P6: track 144.8 -> 174.9 mm
- net P1: track 229.2 -> 254.3 mm
- net P2: track 267.2 -> 286.2 mm, vias 2 -> 0
- net VCC: track 57.2 -> 65.3 mm, vias 0 -> 1
- net P9: track 180.5 -> 172.8 mm, vias 2 -> 0
- net P10: track 166.1 -> 162.2 mm
- net outer_top: track 31.9 -> 31.1 mm
- net ring_home: track 32.1 -> 31.3 mm
- net middle_home: track 32.1 -> 31.3 mm
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Other:
- outline, holes or cut-outs redrawn
- board text added: "Jackalope Keyboard (split) v2.0.1 by @HBBisenieks"
- board text removed: "Jackalope Keyboard (split) v2.0 by @HBBisenieks"
