File: pcb/v2_0/split/split_minimal_case_plate.kicad_pcb (KiCad board)
At the start: 2 copper layers, 172.5 x 116.9 mm, 75 parts

Commit message: split pcb routed, gerbers
Other:
- outline, holes or cut-outs redrawn
Changed lines of the file:
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@@
   (page A3)
   (title_block
-    (title minimal_case_plate)
+    (title split_minimal_case_plate)
     (rev v1.0.0)
     (company Unknown)
@@
 (gr_line (start 140.13932599999998 27.664197499999997) (end 127.55620929999999 21.527001399999996) (angle 90) (layer Edge.Cuts) (width 0.15))
 (gr_line (start 127.55620929999999 21.527001399999996) (end 121.4190132 34.110118099999994) (angle 90) (layer Edge.Cuts) (width 0.15))
-(gr_circle (center 7.303921099999998 -24.5693455) (end 8.303921099999998 -24.5693455) (layer Edge.Cuts) (width 0.15))
-(gr_circle (center 8.2805118 -10.6034488) (end 9.2805118 -10.6034488) (layer Edge.Cuts) (width 0.15))
+(gr_circle (center 6.990016999999998 -29.0583837) (end 7.990016999999998 -29.0583837) (layer Edge.Cuts) (width 0.15))
+(gr_circle (center 8.315389999999999 -10.1046668) (end 9.315389999999999 -10.1046668) (layer Edge.Cuts) (width 0.15))
 (gr_circle (center 47.9249606 -42.3307199) (end 48.9249606 -42.3307199) (layer Edge.Cuts) (width 0.15))
 (gr_circle (center 47.9249606 -23.3307199) (end 48.9249606 -23.3307199) (layer Edge.Cuts) (width 0.15))
